File: HW/KX-T30810/KX-T30810.kicad_sch (KiCad schematic)
At the start: 18 parts, among them IC100 HD63B03XP, IC104 74LS139, IC107 74LS32, U1 4066

Commit message: Schematic
Parts:
- added R916, R917: 2k2, Resistor_SMD:R_0805_2012Metric, symbol Device:R_Small
Changed lines of the file:
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@@
+	)
+	(symbol
+		(lib_id "Device:R_Small")
+		(at 334.01 38.1 0)
+		(unit 1)
+		(exclude_from_sim no)
+		(in_bom yes)
+		(on_board yes)
+		(dnp no)
+		(fields_autoplaced yes)
+		(property "Reference" "R917"
+			(at 336.55 36.8299 0)
+			(effects
+				(font
+					(size 1.016 1.016)
+				)
+				(justify left)
+			)
+		)
+		(property "Value" "2k2"
+			(at 336.55 39.3699 0)
+			(effects
+				(font
+					(size 1.27 1.27)
+				)
+				(justify left)
+			)
+		)
+		(property "Footprint" "Resistor_SMD:R_0805_2012Metric"
+			(at 334.01 38.1 0)
+			(effects
+				(font
+					(size 1.27 1.27)
+				)
+				(hide yes)
+			)
+		)
+		(property "Datasheet" "~"
+			(at 334.01 38.1 0)
+			(effects
+				(font
+					(size 1.27 1.27)
+				)
+				(hide yes)
+			)
+		)
+		(property "Description" "Resistor, small symbol"
+			(at 334.01 38.1 0)
+			(effects
+				(font
+					(size 1.27 1.27)
+				)
+				(hide yes)
+			)
+		)
+		(pin "2"
+		)
+		(pin "1"
+		)
+		(instances
+			(project "KX-T30810"
+				(path "/ec9be23a-b18c-4a96-a888-e3ce388a69ec"
+					(reference "R917")
+					(unit 1)
+				)
+			)
+		)
+	)
+	(symbol
+		(lib_id "Device:R_Small")
+		(at 322.58 38.1 0)
+		(unit 1)
+		(exclude_from_sim no)
+		(in_bom yes)
+		(on_board yes)
+		(dnp no)
+		(fields_autoplaced yes)
+		(property "Reference" "R916"
+			(at 325.12 36.8299 0)
+			(effects
+				(font
+					(size 1.016 1.016)
+				)
+				(justify left)
+			)
+		)
+		(property "Value" "2k2"
+			(at 325.12 39.3699 0)
+			(effects
+				(font
+					(size 1.27 1.27)
+				)
+				(justify left)
+			)
+		)
+		(property "Footprint" "Resistor_SMD:R_0805_2012Metric"
+			(at 322.58 38.1 0)
+			(effects
+				(font
+					(size 1.27 1.27)
+				)
+				(hide yes)
+			)
+		)
+		(property "Datasheet" "~"
+			(at 322.58 38.1 0)
+			(effects
+				(font
+					(size 1.27 1.27)
+				)
+				(hide yes)
+			)
+		)
+		(property "Description" "Resistor, small symbol"
+			(at 322.58 38.1 0)
+			(effects
+				(font
+					(size 1.27 1.27)
+				)
+				(hide yes)
+			)
+		)
+		(pin "2"
+		)
+		(pin "1"
+		)
+		(instances
+			(project ""
+				(path "/ec9be23a-b18c-4a96-a888-e3ce388a69ec"
+					(reference "R916")
+					(unit 1)
+				)
+			)
+		)
 	)
 	(symbol

Commit message: schematic
Parts:
- IC104: footprint (none) -> Package_DIP:CERDIP-16_W7.62mm_SideBrazed
- R110, R111, R112, R113, R114, R115, R116, R117, R133, R134: footprint Resistor_THT:R_Axial_DIN0204_L3.6mm_D1.6mm_P5.08mm_Horizontal -> _mine:R_Axial_L3.6mm_D1.6mm_P4.5mm_Horizontal
Connections:
- net D3: now reaches R114.2
- net D3: now also IC100.55 (D3)
- net ~{RD}: now reaches R134.1
- net ~{RD}: now also IC100.63 (~{RD})
- net ~{WR}: now reaches R133.2
- net ~{WR}: now also IC100.62 (~{WR})
- net D6: now reaches R111.2
- net D6: now also IC100.52 (D6)
- net VCC: now reaches IC100.33 (VCC)
- net A15: now reaches IC100.34 (A15)
- net A15: now also Z102.9 (R8)
- net A14: now reaches IC100.35 (A14)
- net A14: now also Z101.9 (R8)
- net A13: now reaches IC100.36 (A13)
- net A13: now also Z102.8 (R7)
- net A12: now reaches IC100.37 (A12)
- net A12: now also Z101.8 (R7)
- net A11: now reaches IC100.38 (A11)
- net A11: now also Z102.7 (R6)
- net A10: now reaches IC100.39 (A10)
- net A10: now also Z101.7 (R6)
- net A9: now reaches IC100.40 (A9)
- net A9: now also Z102.6 (R5)
- net GND: now reaches IC100.42 (GND)
- net A7: now reaches IC100.43 (A7)
- net A6: now reaches IC100.44 (A6)
- net A5: now reaches IC100.45 (A5)
- net A4: now reaches IC100.46 (A4)
- net A3: now reaches IC100.47 (A3)
- net A2: now reaches IC100.48 (A2)
- net A1: now reaches IC100.49 (A1)
- net A0: now reaches IC100.50 (A0)
- net D7: now reaches IC100.51 (D7)
- net D7: now also R110.2
- net D5: now reaches IC100.53 (D5)
- net D5: now also R112.2
- net D4: now reaches IC100.54 (D4)
- net D4: now also R113.2
- net D2: now reaches IC100.56 (D2)
- net D2: now also R115.2
- net D1: now reaches IC100.57 (D1)
- net D1: now also R116.2
- net D0: now reaches IC100.58 (D0)
- net D0: now also R117.2
